Commit message: Mostly stable gazebo simulation working. Added custom PCD and OC publishers

File: ws/src/hunter_description/description/robot_core.xacro (robot description, xacro)
@@ -154,12 +154,48 @@
     </collision>
   </link>
-  <joint name="trailer_hitch_joint" type="continuous">
-    <parent link="chassis"/>
+  <!-- ===== Spherical hitch emulation ===== -->
+  <xacro:property name="hitch_roll_limit"  value="3.14159"/>  <!-- +/-180° -->
+  <xacro:property name="hitch_pitch_limit" value="3.14159"/>
+  <xacro:property name="hitch_yaw_limit"   value="3.14159"/>
+  <xacro:property name="hitch_damping"     value="30.0"/>     <!-- increase if jittery -->
+  <xacro:property name="hitch_friction"    value="0.5"/>
+  <!-- Rx link at chassis rear center -->
+  <link name="hitch_rx_link">
+    <inertial>
+      <mass value="0.5"/>
+      <inertia ixx="0.001" iyy="0.001" izz="0.001" ixy="0" ixz="0" iyz="0"/>
+    </inertial>
+  </link>
+  <joint name="hitch_rx" type="revolute">
+    <parent link="chassis"/>
+    <child  link="hitch_rx_link"/>
+    <origin xyz="${x_base_to_rear} 0 ${hitch_height}" rpy="0 0 0"/>
+    <axis xyz="1 0 0"/> <!-- roll -->
+    <limit lower="-${hitch_roll_limit}" upper="${hitch_roll_limit}" effort="500.0" velocity="5.0"/>
+    <dynamics damping="${hitch_damping}" friction="${hitch_friction}"/>
+  </joint>
+  <!-- Ry link at the same point -->
+  <link name="hitch_ry_link">
+    <inertial>
+      <mass value="0.5"/>
+      <inertia ixx="0.001" iyy="0.001" izz="0.001" ixy="0" ixz="0" iyz="0"/>
+    </inertial>
+  </link>
+  <joint name="hitch_ry" type="revolute">
+    <parent link="hitch_rx_link"/>
+    <child  link="hitch_ry_link"/>
+    <origin xyz="0 0 0" rpy="0 0 0"/>
+    <axis xyz="0 1 0"/> <!-- pitch -->
+    <limit lower="-${hitch_pitch_limit}" upper="${hitch_pitch_limit}" effort="500.0" velocity="5.0"/>
+    <dynamics damping="${hitch_damping}" friction="${hitch_friction}"/>
+  </joint>
+  <!-- Rz joint into your existing trailer_hitch_link (acts like old yaw) -->
+  <joint name="hitch_rz" type="revolute">
+    <parent link="hitch_ry_link"/>
     <child  link="trailer_hitch_link"/>
-    <!-- rear center of chassis, at your defined hitch height -->
-    <origin xyz="${x_base_to_rear} 0 ${hitch_height}" rpy="0 0 0"/>
-    <axis xyz="0 0 1"/>
-    <dynamics damping="0.2" friction="0.5"/>
-    <limit effort="20.0" velocity="50.0"/>
+    <origin xyz="0 0 0" rpy="0 0 0"/>
+    <axis xyz="0 0 1"/> <!-- yaw -->
+    <limit lower="-${hitch_yaw_limit}" upper="${hitch_yaw_limit}" effort="500.0" velocity="5.0"/>
+    <dynamics damping="${hitch_damping}" friction="${hitch_friction}"/>
   </joint>
   <!-- ========== Trailer chassis (frame at ground via drawbar drop) ========== -->
@@ -217,16 +253,16 @@
   </joint>
   <xacro:gazebo_friction reference="trailer_right_wheel"/>
-    <gazebo reference="trailer_left_wheel">
-      <mu1>1.2</mu1>      <!-- along fdir1 (rolling) -->
-      <mu2>0.15</mu2>     <!-- lateral slip allowed -->
-      <slip1>0.0</slip1>  <!-- rolling -->
-      <slip2>0.02</slip2> <!-- lateral relaxation -->
-      <fdir1>1 0 0</fdir1>
-      <kp>2e6</kp> <kd>1e3</kd> <!-- softer contact helps stability -->
-    </gazebo>
-    <gazebo reference="trailer_right_wheel">
-      <mu1>1.2</mu1><mu2>0.15</mu2><slip1>0.0</slip1><slip2>0.02</slip2>
-      <fdir1>1 0 0</fdir1>
-      <kp>2e6</kp> <kd>1e3</kd>
-    </gazebo>
+    <!-- trailer_base_link at axle center (child of trailer_chassis) -->
+    <link name="trailer_base_link">
+      <!-- keep it nearly massless but non-zero for stability -->
+      <inertial>
+        <mass value="0.001"/>
+        <inertia ixx="1e-6" iyy="1e-6" izz="1e-6" ixy="0" ixz="0" iyz="0"/>
+      </inertial>
+    </link>
+    <joint name="trailer_base_fixed" type="fixed">
+      <parent link="trailer_chassis"/>
+      <child  link="trailer_base_link"/>
+      <origin xyz="${trailer_axle_x} 0 ${trailer_wheel_radius}" rpy="0 0 0"/>
+    </joint>
 </robot>

File: ws/src/hunter_description/description/ros2_control.xacro (robot description, xacro)
@@ -33,4 +33,33 @@
       <state_interface name="position"/>
     </joint>
+    <joint name="hitch_rx">
+    <state_interface name="position"/>
+    <state_interface name="velocity"/>
+  </joint>
+  <joint name="hitch_ry">
+    <state_interface name="position"/>
+    <state_interface name="velocity"/>
+  </joint>
+  <joint name="hitch_rz">
+    <state_interface name="position"/>
+    <state_interface name="velocity"/>
+  </joint>
+  <joint name="rear_left_susp_joint">
+    <state_interface name="position"/>
+    <state_interface name="velocity"/>
+  </joint>
+  <joint name="rear_right_susp_joint">
+    <state_interface name="position"/>
+    <state_interface name="velocity"/>
+  </joint>
+  <!-- Trailer wheel spin joints, if you want their states too -->
+  <joint name="trailer_left_wheel_joint">
+    <state_interface name="position"/>
+    <state_interface name="velocity"/>
+  </joint>
+  <joint name="trailer_right_wheel_joint">
+    <state_interface name="position"/>
+    <state_interface name="velocity"/>
+  </joint>
   </ros2_control>
   <gazebo>

Commit message: Added ground truth odometry publisher, stabilized trailer dynamics by tuning rear suspension joint

File: ws/src/hunter_description/description/robot_core.xacro (robot description, xacro)
@@ -32,6 +32,6 @@
     <origin xyz="${x_base_to_rear} ${y_base_to_wheel} ${z_base_to_wheel}" rpy="0 0 0"/>
     <axis xyz="0 0 1"/>
-    <!-- ~6 cm travel, biased slightly upward so static load compresses downward -->
-    <limit lower="-0.05" upper="0.02" effort="1e6" velocity="1.0"/>
+    <!-- 4 cm travel, biased slightly upward so static load compresses downward -->
+    <limit lower="-0.03" upper="0.01" effort="1e6" velocity="1.0"/>
     <dynamics damping="300.0" friction="5.0"/>
   </joint>
@@ -61,5 +61,5 @@
     <origin xyz="${x_base_to_rear} -${y_base_to_wheel} ${z_base_to_wheel}" rpy="0 0 0"/>
     <axis xyz="0 0 1"/>
-    <limit lower="-0.05" upper="0.02" effort="1e6" velocity="1.0"/>
+    <limit lower="-0.03" upper="0.01" effort="1e6" velocity="1.0"/>
     <dynamics damping="300.0" friction="5.0"/>
   </joint>
@@ -124,7 +124,7 @@
   </joint>
   <!-- ===== Trailer params (tweak as needed) ===== -->
-  <xacro:property name="trailer_length"         value="5.0"/>
+  <xacro:property name="trailer_length"         value="3.5"/>
   <xacro:property name="trailer_width"          value="0.8"/>
-  <xacro:property name="trailer_height"         value="1.2"/>
+  <xacro:property name="trailer_height"         value="0.8"/>
   <xacro:property name="trailer_mass"           value="100.0"/>
   <xacro:property name="hitch_height"           value="0.0"/>
@@ -132,6 +132,6 @@
   <xacro:property name="trailer_wheel_radius"   value="${z_base_to_wheel}"/>
   <xacro:property name="trailer_clearance"      value="0.05"/>   <!-- gap box bottom ↔ tire top -->
-  <xacro:property name="trailer_axle_from_rear" value="0.6"/>    <!-- axle forward from rear bumper -->
-  <xacro:property name="trailer_drawbar_len"    value="2.75"/>    <!-- hitch → chassis frame along -X -->
+  <xacro:property name="trailer_axle_from_rear" value="0.3"/>    <!-- axle forward from rear bumper -->
+  <xacro:property name="trailer_drawbar_len"    value="1.75"/>    <!-- hitch → chassis frame along -X -->
   <!-- Derived positions (chassis frame at ground z=0 via drawbar offset) -->
   <xacro:property name="trailer_axle_x" value="${-trailer_length/2.0 + trailer_axle_from_rear}"/>
@@ -155,11 +155,10 @@
   </link>
   <!-- ===== Spherical hitch emulation ===== -->
-  <xacro:property name="hitch_roll_limit"  value="3.14159"/>  <!-- +/-180° -->
-  <xacro:property name="hitch_pitch_limit" value="3.14159"/>
-  <xacro:property name="hitch_yaw_limit"   value="3.14159"/>
-  <xacro:property name="hitch_damping"     value="30.0"/>     <!-- increase if jittery -->
+  <xacro:property name="hitch_pitch_limit" value="0.1"/>
+  <xacro:property name="hitch_yaw_limit"   value="1.3"/>
+  <xacro:property name="hitch_damping"     value="30.0"/>
   <xacro:property name="hitch_friction"    value="0.5"/>
-  <!-- Rx link at chassis rear center -->
-  <link name="hitch_rx_link">
+  <!-- Ry link at the same point -->
+  <link name="hitch_ry_link">
     <inertial>
       <mass value="0.5"/>
@@ -167,21 +166,6 @@
     </inertial>
   </link>
-  <joint name="hitch_rx" type="revolute">
-    <parent link="chassis"/>
-    <child  link="hitch_rx_link"/>
-    <origin xyz="${x_base_to_rear} 0 ${hitch_height}" rpy="0 0 0"/>
-    <axis xyz="1 0 0"/> <!-- roll -->
-    <limit lower="-${hitch_roll_limit}" upper="${hitch_roll_limit}" effort="500.0" velocity="5.0"/>
-    <dynamics damping="${hitch_damping}" friction="${hitch_friction}"/>
-  </joint>
-  <!-- Ry link at the same point -->
-  <link name="hitch_ry_link">
-    <inertial>
-      <mass value="0.5"/>
-      <inertia ixx="0.001" iyy="0.001" izz="0.001" ixy="0" ixz="0" iyz="0"/>
-    </inertial>
-  </link>
   <joint name="hitch_ry" type="revolute">
-    <parent link="hitch_rx_link"/>
+    <parent link="chassis"/>
     <child  link="hitch_ry_link"/>
     <origin xyz="0 0 0" rpy="0 0 0"/>
@@ -266,3 +250,15 @@
       <origin xyz="${trailer_axle_x} 0 ${trailer_wheel_radius}" rpy="0 0 0"/>
     </joint>
+    <gazebo>
+      <plugin name="gt_odom" filename="libgazebo_ros_p3d.so">
+        <!-- TF frames -->
+        <frame_name>odom</frame_name>
+        <body_name>base_link</body_name>
+        <publish_tf>true</publish_tf>
+        <update_rate>50.0</update_rate>
+        <gaussian_noise>0.0</gaussian_noise>
+        <xyz_offset>0 0 0</xyz_offset>
+        <rpy_offset>0 0 0</rpy_offset>
+      </plugin>
+    </gazebo>
 </robot>

Commit message: commit for test on Mar 3 2026

File: ws/src/hunter_description/description/robot_core.xacro (robot description, xacro)
@@ -4,10 +4,5 @@
   <xacro:include filename="inertial_macros.xacro"/>
   <xacro:include filename="meshes.xacro"/>
-  <!-- Constants for robot dimensions -->
-  <xacro:property name="z_base_to_wheel" value="-0.19558" />
-  <xacro:property name="x_base_to_rear" value="-0.28" />
-  <xacro:property name="x_base_to_front" value="0.37142" />
-  <xacro:property name="y_base_to_wheel" value="0.2925" />
-  <xacro:property name="max_steer_angle_central" value="0.461" />
+  <xacro:include filename="common.xacro"/>
   <link name="base_link"/>
   <joint name="chassis_joint" type="fixed">
@@ -123,131 +118,4 @@
     <axis   xyz="0 0 -1" />
   </joint>
-  <!-- ===== Trailer params (tweak as needed) ===== -->
-  <xacro:property name="trailer_length"         value="3.5"/>
-  <xacro:property name="trailer_width"          value="0.8"/>
-  <xacro:property name="trailer_height"         value="0.8"/>
-  <xacro:property name="trailer_mass"           value="100.0"/>
-  <xacro:property name="hitch_height"           value="0.0"/>
-  <!-- match your robot’s wheel radius if you want identical tire size -->
-  <xacro:property name="trailer_wheel_radius"   value="${z_base_to_wheel}"/>
-  <xacro:property name="trailer_clearance"      value="0.05"/>   <!-- gap box bottom ↔ tire top -->
-  <xacro:property name="trailer_axle_from_rear" value="0.3"/>    <!-- axle forward from rear bumper -->
-  <xacro:property name="trailer_drawbar_len"    value="1.75"/>    <!-- hitch → chassis frame along -X -->
-  <!-- Derived positions (chassis frame at ground z=0 via drawbar offset) -->
-  <xacro:property name="trailer_axle_x" value="${-trailer_length/2.0 + trailer_axle_from_rear}"/>
-  <xacro:property name="trailer_axle_z" value="${trailer_wheel_radius}"/>
-  <xacro:property name="trailer_box_z"  value="${trailer_height/2.0 + trailer_wheel_radius + trailer_clearance}"/>
-  <xacro:property name="trailer_box_z"  value="${trailer_height/2.0 + trailer_clearance}"/>
-  <!-- ========== Hitch pivot at chassis rear (yaw about Z) ========== -->
-  <link name="trailer_hitch_link">
-    <inertial>
-      <mass value="5.0"/>
-      <inertia ixx="0.02" iyy="0.02" izz="0.02" ixy="0" ixz="0" iyz="0"/>
-    </inertial>
-    <visual>
-      <geometry><cylinder radius="0.04" length="0.12"/></geometry>
-      <origin xyz="0 0 0"/>
-      <material name="dark_grey"><color rgba="0.2 0.2 0.2 1"/></material>
-    </visual>
-    <collision>
-      <geometry><cylinder radius="0.04" length="0.12"/></geometry>
-    </collision>
-  </link>
-  <!-- ===== Spherical hitch emulation ===== -->
-  <xacro:property name="hitch_pitch_limit" value="0.1"/>
-  <xacro:property name="hitch_yaw_limit"   value="1.3"/>
-  <xacro:property name="hitch_damping"     value="30.0"/>
-  <xacro:property name="hitch_friction"    value="0.5"/>
-  <!-- Ry link at the same point -->
-  <link name="hitch_ry_link">
-    <inertial>
-      <mass value="0.5"/>
-      <inertia ixx="0.001" iyy="0.001" izz="0.001" ixy="0" ixz="0" iyz="0"/>
-    </inertial>
-  </link>
-  <joint name="hitch_ry" type="revolute">
-    <parent link="chassis"/>
-    <child  link="hitch_ry_link"/>
-    <origin xyz="0 0 0" rpy="0 0 0"/>
-    <axis xyz="0 1 0"/> <!-- pitch -->
-    <limit lower="-${hitch_pitch_limit}" upper="${hitch_pitch_limit}" effort="500.0" velocity="5.0"/>
-    <dynamics damping="${hitch_damping}" friction="${hitch_friction}"/>
-  </joint>
-  <!-- Rz joint into your existing trailer_hitch_link (acts like old yaw) -->
-  <joint name="hitch_rz" type="revolute">
-    <parent link="hitch_ry_link"/>
-    <child  link="trailer_hitch_link"/>
-    <origin xyz="0 0 0" rpy="0 0 0"/>
-    <axis xyz="0 0 1"/> <!-- yaw -->
-    <limit lower="-${hitch_yaw_limit}" upper="${hitch_yaw_limit}" effort="500.0" velocity="5.0"/>
-    <dynamics damping="${hitch_damping}" friction="${hitch_friction}"/>
-  </joint>
-  <!-- ========== Trailer chassis (frame at ground via drawbar drop) ========== -->
-  <link name="trailer_chassis">
-    <inertial>
-      <mass value="${trailer_mass}"/>
-      <inertia
-        ixx="${(1/12.0)*trailer_mass*(trailer_height*trailer_height + trailer_length*trailer_length)}"
-        iyy="${(1/12.0)*trailer_mass*(trailer_width*trailer_width  + trailer_length*trailer_length)}"
-        izz="${(1/12.0)*trailer_mass*(trailer_width*trailer_width  + trailer_height*trailer_height)}"
-        ixy="0" ixz="0" iyz="0"/>
-    </inertial>
-    <!-- Visual box sits above tires -->
-    <visual>
-      <geometry><box size="${trailer_length} ${trailer_width} ${trailer_height}"/></geometry>
-      <origin xyz="0 0 ${trailer_box_z}" rpy="0 0 0"/>
-      <material name="trailergrey"><color rgba="0.75 0.75 0.75 1"/></material>
-    </visual>
-    <collision>
-      <geometry><box size="${trailer_length} ${trailer_width} ${trailer_height}"/></geometry>
-      <origin xyz="0 0 ${trailer_box_z}" rpy="0 0 0"/>
-    </collision>
-  </link>
-  <!-- Fix trailer frame w.r.t. hitch and drop to ground by hitch_height -->
-  <joint name="trailer_drawbar_joint" type="fixed">
-    <parent link="trailer_hitch_link"/>
-    <child  link="trailer_chassis"/>
-    <origin xyz="-${trailer_drawbar_len} 0 -${hitch_height}" rpy="0 0 0"/>
-  </joint>
-  <!-- ========== Wheels (reuse your robot’s wheel meshes/inertials) ========== -->
-  <link name="trailer_left_wheel">
-    <xacro:mesh name="rear_left_wheel"/>
-    <xacro:inertial_wheel/>
-  </link>
-  <joint name="trailer_left_wheel_joint" type="continuous">
-    <parent link="trailer_chassis"/>
-    <child  link="trailer_left_wheel"/>
-    <origin xyz="${trailer_axle_x} ${trailer_width/2.0} ${trailer_axle_z}" rpy="${pi/2} 0 0"/>
-    <axis xyz="0 0 -1"/>
-    <dynamics damping="0.2" friction="0.5"/>
-    <limit effort="20.0" velocity="50.0"/>
-  </joint>
-  <xacro:gazebo_friction reference="trailer_left_wheel"/>
-  <link name="trailer_right_wheel">
-    <xacro:mesh name="rear_right_wheel"/>
-    <xacro:inertial_wheel/>
-  </link>
-  <joint name="trailer_right_wheel_joint" type="continuous">
-    <parent link="trailer_chassis"/>
-    <child  link="trailer_right_wheel"/>
-    <origin xyz="${trailer_axle_x} -${trailer_width/2.0} ${trailer_axle_z}" rpy="${pi/2} 0 0"/>
-    <axis xyz="0 0 -1"/>
-    <dynamics damping="0.2" friction="0.5"/>
-    <limit effort="20.0" velocity="50.0"/>
-  </joint>
-  <xacro:gazebo_friction reference="trailer_right_wheel"/>
-    <!-- trailer_base_link at axle center (child of trailer_chassis) -->
-    <link name="trailer_base_link">
-      <!-- keep it nearly massless but non-zero for stability -->
-      <inertial>
-        <mass value="0.001"/>
-        <inertia ixx="1e-6" iyy="1e-6" izz="1e-6" ixy="0" ixz="0" iyz="0"/>
-      </inertial>
-    </link>
-    <joint name="trailer_base_fixed" type="fixed">
-      <parent link="trailer_chassis"/>
-      <child  link="trailer_base_link"/>
-      <origin xyz="${trailer_axle_x} 0 ${trailer_wheel_radius}" rpy="0 0 0"/>
-    </joint>
     <gazebo>
       <plugin name="gt_odom" filename="libgazebo_ros_p3d.so">
